File: ADS1115_Featherwing.brd (EAGLE design)
At the start: 50.8 x 22.9 mm, 24 parts, among them J2 ST-PJ-312, U1 ADS1115IDGST

Commit message: Rewired fixed board
Parts:
- moved U$7 13.9 mm to (38.3, 3.89), turned to 90 degrees
Connections:
- net N$4: now also U$7.1; no longer U$7.3
- net REOUT: now also U$7.3; no longer U$7.1
Routing:
- net GND: track 60.0 -> 0.03 mm, vias 15 -> 24
- net ALERT: track 34.6 -> 19.1 mm
- net AIN3: track 26.9 -> 38.8 mm, vias 5 -> 1
- net AIN1: track 38.1 -> 27.2 mm, vias 3 -> 1
- net N$4: track 23.6 -> 13.5 mm, vias 2 -> 0
- net SCL: track 37.4 -> 27.8 mm
- net VDD: track 42.9 -> 48.9 mm, vias 0 -> 2
- net SDA: track 42.8 -> 36.9 mm, vias 4 -> 2
- net N$3: track 21.1 -> 26.4 mm
- net AIN0: track 44.4 -> 49.6 mm, vias 3 -> 1
- net REOUT: track 26.9 -> 24.2 mm, vias 2 -> 0
- net N$2: track 4.70 -> 2.74 mm, vias 2 -> 0
- net AIN2: track 24.2 -> 25.6 mm
- net ADDR: track 45.5 -> 44.7 mm
Other:
- board text added: "3V3"
- board text added: "@whatnick 17/01/2016 v2"
- board text added: "GND"
- board text added: "SCL"
- board text added: "SDA"
- board text added: "VUSB"
- board text removed: "@whatnick 26/12/2015 v1"

Commit message: Added grove connector
Parts:
- added J1: 4P-SMD-2.0-90D, Seeed-OPL-Connector:HW4-SMD-2.0-90D
- moved 0X4A 13.2 mm to (26.9, 5.08), turned to 90 degrees
- moved 0X4B 12.9 mm to (35.6, 5.08), turned to 90 degrees
- moved 0X49 12.2 mm to (29.7, 5.08), turned to 270 degrees
- moved 0X48 9.16 mm to (32.7, 5.08), turned to 270 degrees
- moved C1 4.58 mm to (35.4, 11.3)
- moved U1 4.25 mm to (32.4, 11.4)
- moved U$7 1.27 mm to (37.0, 3.89)
Connections:
- removed net N$1: C2.1, FB1.1
- removed net N$2: C2.2, FB2.1
- new net 3V: C2.1, FB1.1, J1.3, MS1.2
- new net AGND: B2.-, C2.2, C3.2, C4.2, FB2.1, J1.4, MS1.4, U$7.2
- net GND: now also J1.SS1, J1.SS2; no longer B2.-, C3.2, C4.2, MS1.4, U$7.2
- net SCL: now also J1.1
- net SDA: now also J1.2
- net VDD: no longer MS1.2
Routing:
- net AGND: track 0.00 -> 45.5 mm, vias 0 -> 2
- net 3V: track 0.00 -> 39.7 mm, vias 0 -> 3
- net ADDR: track 44.7 -> 21.1 mm, vias 0 -> 3
- net AIN3: track 38.8 -> 60.1 mm, vias 1 -> 6
- net VDD: track 48.9 -> 27.6 mm, vias 2 -> 0
- net SCL: track 27.8 -> 44.9 mm, vias 4 -> 2
- net AIN0: track 49.6 -> 37.6 mm, vias 1 -> 4
- net GND: track 0.03 -> 11.5 mm, vias 24 -> 19
- net AIN1: track 27.2 -> 38.4 mm
- net SDA: track 36.9 -> 42.3 mm, vias 2 -> 3
- net N$3: track 26.4 -> 21.1 mm
- net ALERT: track 19.1 -> 16.2 mm
- net N$1: track 2.75 -> 0.00 mm
- net N$2: track 2.74 -> 0.00 mm
- net AIN2: track 25.6 -> 23.1 mm, vias 1 -> 3
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
Commit message: Switched to 50V electrolytic
Parts:
- removed C3: 100uF, adafruit:C1210
- added C5: 100uF 50V, adafruit:153CLV-0810
- C4: value 10uF -> 10uF 50V
- moved C1 16.9 mm to (20.2, 18.8), turned to 180 degrees
- moved C4 14.5 mm to (20.7, 19.1), turned to 180 degrees
- moved U1 12.6 mm to (20.4, 15.3), turned to 270 degrees
- moved D2 7.70 mm to (28.0, 19.4), turned to 180 degrees
- moved R7 6.81 mm to (8.00, 20.3), turned to 180 degrees
- moved R6 4.67 mm to (12.4, 20.3), turned to 180 degrees
- moved B2 4.47 mm to (20.4, 14.6)
- moved U$7 2.52 mm to (39.3, 4.95)
Connections:
- net AGND: now also C5.-; no longer C3.2
- net N$4: now also C5.+; no longer C4.1
- net REOUT: now also C4.1; no longer C3.1
Routing:
- net GND: track 11.5 -> 68.5 mm, vias 19 -> 20
- net AIN2: track 23.1 -> 58.4 mm, vias 3 -> 1
- net SDA: track 42.3 -> 65.5 mm, vias 3 -> 2
- net AIN1: track 38.4 -> 20.3 mm
- net AIN0: track 37.6 -> 26.6 mm, vias 4 -> 1
- net ADDR: track 21.1 -> 31.7 mm, vias 3 -> 2
- net SCL: track 44.9 -> 53.3 mm
- net ALERT: track 16.2 -> 8.31 mm, vias 2 -> 0
- net AGND: track 45.5 -> 52.2 mm, vias 2 -> 3
- net AIN3: track 60.1 -> 55.9 mm, vias 6 -> 3
- net REOUT: track 21.9 -> 18.3 mm
- net USB: track 2.69 -> 5.70 mm
- net N$4: track 13.1 -> 10.5 mm
- net 3V: track 39.7 -> 41.6 mm
- net N$3: track 21.1 -> 22.6 mm, vias 0 -> 2
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
Commit message: Added protection resistor
Parts:
- added R8: 10K, resistor:R0603
- moved R6 1.13 mm to (12.2, 21.4)
- moved R7 1.12 mm to (8.10, 21.4)
Connections:
- new net N$1: R8.2, U1.5
- net AIN1: now also R8.1; no longer U1.5
Routing:
- net GND: track 68.5 -> 31.5 mm, vias 20 -> 13
- net AIN1: track 20.3 -> 4.18 mm, vias 1 -> 0
- net N$1: track 0.00 -> 16.0 mm, vias 0 -> 1
- net SDA: track 65.5 -> 79.9 mm, vias 2 -> 4
- net AIN2: track 58.4 -> 61.7 mm, vias 1 -> 3
- net AGND: track 52.2 -> 50.1 mm, vias 3 -> 1
- net AIN0: track 26.6 -> 27.6 mm
- net N$3: track 22.6 -> 23.5 mm

Commit message: Switched to XP Power Vreg
Parts:
- removed U$7: ROF-78E, recom-intl:SMD-4
- added U2: SR05, Seeed-OPL-ic:SR05
- C4: value 10uF 50V -> 10uF; device adafruit:C1206 -> adafruit:153CLV-0405
- moved C4 8.84 mm to (28.1, 14.4), turned to 90 degrees
- moved 0X4A 0.41 mm to (26.5, 5.08), turned to 270 degrees
- moved 0X4B 0.05 mm to (35.5, 5.08), turned to 270 degrees
- renumbered C5 to C3
Connections:
- removed net REOUT: C4.1, D2.+, U$7.3
- new net N$2: C4.+, D2.+, U2.P$3
- net AGND: now also C4.-, U2.P$2; no longer C4.2, U$7.2
- net N$4: now also U2.P$1; no longer U$7.1
Routing:
- net VDD: track 28.5 -> 53.3 mm, vias 0 -> 2
- net AIN2: track 61.7 -> 38.5 mm
- net N$4: track 10.5 -> 32.7 mm, vias 0 -> 2
- net REOUT: track 18.3 -> 0.00 mm
- net N$2: track 0.00 -> 14.6 mm, vias 0 -> 1
- net SDA: track 79.9 -> 71.4 mm
- net ADDR: track 31.7 -> 23.3 mm, vias 2 -> 0
- net AIN3: track 55.5 -> 62.6 mm
- net AGND: track 50.1 -> 43.8 mm
- net GND: track 31.5 -> 26.5 mm, vias 13 -> 11
- net AIN0: track 27.6 -> 23.7 mm
- net 3V: track 41.6 -> 43.9 mm, vias 3 -> 2
- net N$1: track 16.0 -> 13.9 mm
- net SCL: track 53.3 -> 51.4 mm
- net ALERT: track 8.31 -> 9.72 mm, vias 0 -> 2

Commit message: Renumber parts/reversion
Parts:
- removed J4: (no value), dp_devices:DC_BARREL_JACK_SMD_2MM
- added J3: 4P-SMD-2.0-90D, Seeed-OPL-Connector:HW4-SMD-2.0-90D
- C1: value 1µF -> 10uF; device microbuilder:0603 -> adafruit:153CLV-0405
- C2: value 1µF -> 100uF 50V; device microbuilder:0603 -> adafruit:153CLV-0810
- C3: value 100uF 50V -> 1µF; device adafruit:153CLV-0810 -> microbuilder:0603
- C4: value 10uF -> 1µF; device adafruit:153CLV-0405 -> microbuilder:0603
- J1: value 4P-SMD-2.0-90D -> (none); device Seeed-OPL-Connector:HW4-SMD-2.0-90D -> dp_devices:DC_BARREL_JACK_SMD_2MM
- R1: value 10K -> 100K; device microbuilder:0603 -> resistor:R0603
- R2: device microbuilder:0603 -> resistor:R0603
- R5: value 100R -> 10K
- R6: value 100K -> 100R; device resistor:R0603 -> microbuilder:0603
- R8: device resistor:R0603 -> microbuilder:0603
- U1: value ADS1115IDGST -> SR05; device microbuilder:MSOP10 -> Seeed-OPL-ic:SR05
- U2: value SR05 -> ADS1115IDGST; device Seeed-OPL-ic:SR05 -> microbuilder:MSOP10
- moved R6 31.0 mm to (43.2, 19.1), turned to 0 degrees
- moved J1 31.0 mm to (7.62, 11.4), flipped to the top, turned to 270 degrees
- moved R5 23.9 mm to (21.6, 8.89), flipped to the bottom, turned to 90 degrees
- moved R2 22.4 mm to (8.10, 21.4), flipped to the top, turned to 180 degrees
- moved R1 21.1 mm to (12.2, 21.4), flipped to the top, turned to 180 degrees
- moved R8 16.1 mm to (24.1, 8.89), flipped to the bottom, turned to 90 degrees
- moved C4 13.5 mm to (17.8, 5.71), flipped to the bottom, turned to 0 degrees
- moved C3 11.7 mm to (20.2, 18.8), flipped to the bottom, turned to 180 degrees
- moved U1 11.6 mm to (31.8, 17.8), flipped to the top
- moved U2 11.6 mm to (20.4, 15.3), flipped to the bottom
- moved C1 9.08 mm to (28.1, 14.4), flipped to the top, turned to 90 degrees
- moved R3 5.08 mm to (29.2, 8.89)
- moved R4 5.08 mm to (26.7, 8.89)
- moved R7 4.49 mm to (12.2, 19.7), turned to 0 degrees
- moved C2 3.55 mm to (21.0, 7.14), flipped to the top
- renumbered 0X48 to 0X1, 0X49 to 0X2, B2 to B1, D2 to D1
Connections:
- net 3V: now also C4.1, J3.3; no longer C2.1, J1.3
- net ADDR: now also R8.1, U2.1; no longer R3.1, U1.1
- net AGND: now also C1.-, C2.-, C4.2, J3.4, U1.P$2; no longer C2.2, C3.-, C4.-, J1.4, U2.P$2
- net AIN0: now also J1.P1@2, R2.2, U2.4; no longer J4.P1@2, R7.2, U1.4
- net AIN1: now also R1.2, R2.1; no longer R6.2, R8.1
- net AIN2: now also R6.1, U2.6; no longer R5.1, U1.6
- net AIN3: now also R6.2, U2.7; no longer R5.2, U1.7
- net ALERT: now also R5.2, U2.2; no longer R4.2, U1.2
- net GND: now also C3.1, J3.SS1, J3.SS2, R8.2, U2.3; no longer C1.1, J1.SS1, J1.SS2, R3.2, U1.3
- net N$1: now also R7.2, U2.5; no longer R8.2, U1.5
- net N$2: now also C1.+, U1.P$3; no longer C4.+, U2.P$3
- net N$3: now also J1.P2, R1.1; no longer J4.P2, R6.1
- net N$4: now also C2.+, U1.P$1; no longer C3.+, U2.P$1
- net SCL: now also J3.1, R3.2, U2.10; no longer J1.1, R1.2, U1.10
- net SDA: now also J3.2, R4.2, U2.9; no longer J1.2, R2.2, U1.9
- net VDD: now also C3.2, R3.1, R5.1, U2.8; no longer C1.2, R1.1, R2.1, U1.8
Other:
- board text added: "@whatnick 18/02/2016 v3"
- board text removed: "@whatnick 17/01/2016 v2"
