File: ADS1115_Featherwing.brd (EAGLE design)
At the start: 50.8 x 22.9 mm, 26 parts, among them J2 ST-PJ-312, J3 4P-SMD-2.0-90D, U1 SR05, U2 ADS1115IDGST

Commit message: Rewired with better net names
Parts:
- R7: device resistor:R0603 -> microbuilder:0603
- moved C3 7.79 mm to (28.0, 18.0)
- moved U2 7.47 mm to (27.9, 15.2), turned to 90 degrees
- moved R7 4.86 mm to (17.0, 18.8), turned to 180 degrees
- moved R2 0.97 mm to (8.03, 20.5)
- moved R1 0.97 mm to (12.3, 20.5)
- moved U1 0.86 mm to (31.0, 17.4)
- moved C1 0.56 mm to (27.6, 14.3)
- moved C2 0.07 mm to (21.0, 7.09), turned to 180 degrees
- renumbered 0X1 to 0X48, 0X2 to 0X49
Connections:
- removed net AIN0: B1.~2, J1.P1@2, R2.2, U2.4
- removed net AIN1: R1.2, R2.1, R7.1
- removed net AIN2: J2.COM1, R6.1, U2.6
- removed net AIN3: J2.L, R6.2, U2.7
- new net I_AC+: J2.COM1, R6.1, U2.4
- new net I_AC-: J2.L, R6.2, U2.5
- new net V_AC+: R1.2, R2.1, U2.7
- new net V_AC-: B1.~2, J1.P1@2, R2.2, R7.1
- net AGND: now also J3.SS1, J3.SS2
- net GND: no longer J3.SS1, J3.SS2
- net N$1: now also U2.6; no longer U2.5
Routing:
- net AIN3: track 62.6 -> 0.00 mm, vias 3 -> 0
- net I_AC-: track 0.00 -> 53.2 mm, vias 0 -> 3
- net AIN2: track 38.5 -> 0.00 mm, vias 3 -> 0
- net AGND: track 43.8 -> 80.7 mm, vias 1 -> 19
- net I_AC+: track 0.00 -> 31.1 mm, vias 0 -> 1
- net V_AC+: track 0.00 -> 29.0 mm, vias 0 -> 1
- net V_AC-: track 0.00 -> 24.8 mm
- net AIN0: track 23.7 -> 0.00 mm, vias 1 -> 0
- net VDD: track 53.3 -> 29.7 mm, vias 2 -> 0
- net SCL: track 51.4 -> 36.0 mm
- net SDA: track 71.4 -> 57.4 mm, vias 4 -> 2
- net N$4: track 32.7 -> 22.7 mm, vias 2 -> 1
- net GND: track 26.5 -> 36.4 mm, vias 11 -> 2
- net N$1: track 13.9 -> 23.3 mm, vias 1 -> 3
- net 3V: track 43.9 -> 53.1 mm, vias 2 -> 0
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- added copper zone on layer 1, net AGND
- added copper zone on layer 16, net AGND
- removed copper zone on layer 1, net GND
- removed copper zone on layer 16, net GND

Commit message: Added clamper and power LED
Parts:
- added C5, C6, C7, C8: 33nF, microbuilder:0603
- added PWR: GREEN, Discrete-new:LED-0603
- added R10, R13, R9: 1K, microbuilder:0603
- added R11: 10K, microbuilder:0603
- added R12: VARISTORCN0603, varistor:CT/CN0603
- added R14: 1k, Discrete-new:R0603
- R7: value 10K -> 1K
- R8: value 10K -> VARISTORCN0603; device microbuilder:0603 -> varistor:CT/CN0603
- moved R8 9.86 mm to (18.6, 17.1)
- moved C3 5.44 mm to (22.6, 17.4)
- moved U2 5.23 mm to (22.7, 14.7)
- moved D1 2.11 mm to (25.9, 19.3)
- moved R7 1.80 mm to (16.4, 17.1), flipped to the bottom, turned to 270 degrees
Connections:
- new net N$5: C5.1, R7.2, R8.1, U2.4
- new net N$6: C7.1, R10.2, R12.1, U2.6
- new net N$7: C8.2, R12.2, R13.2, U2.7
- new net N$8: PWR.+, R14.2
- net ADDR: now also R11.1; no longer R8.1
- net AGND: now also PWR.-
- net GND: now also C5.2, C6.1, C7.2, C8.1, R11.2; no longer R8.2
- net I_AC+: now also R10.1; no longer U2.4
- net I_AC-: now also R13.1; no longer U2.5
- net N$1: now also C6.2, R8.2, R9.2, U2.5; no longer R7.2, U2.6
- net USB: now also R14.1
- net V_AC+: now also R7.1; no longer U2.7
- net V_AC-: now also R9.1; no longer R7.1
Routing:
- net AGND: track 80.7 -> 48.8 mm, vias 19 -> 23
- net N$7: track 0.00 -> 18.8 mm, vias 0 -> 2
- net GND: track 36.4 -> 54.6 mm, vias 2 -> 0
- net I_AC-: track 53.2 -> 39.0 mm, vias 3 -> 1
- net 3V: track 53.1 -> 38.9 mm, vias 0 -> 2
- net V_AC+: track 29.0 -> 15.8 mm
- net N$1: track 23.3 -> 12.5 mm, vias 3 -> 2
- net N$6: track 0.00 -> 10.4 mm
- net I_AC+: track 31.1 -> 23.3 mm
- net ALERT: track 13.3 -> 5.66 mm, vias 2 -> 0
- net SDA: track 57.4 -> 50.7 mm, vias 2 -> 4
- net N$5: track 0.00 -> 6.42 mm
- net V_AC-: track 24.8 -> 19.0 mm, vias 0 -> 1
- net SCL: track 36.0 -> 41.6 mm, vias 2 -> 4
- net N$3: track 22.6 -> 27.7 mm, vias 2 -> 0
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Other:
- board text added: "@whatnick 21/02/2016 v3"
- board text removed: "@whatnick 18/02/2016 v3"

Commit message: Reposition parts
Parts:
- R1: value 100K -> 120K
Routing:
- net AGND: vias 23 -> 25
Other:
- board text added: "whatnick 21/02/2016 v3"
- board text removed: "@whatnick 21/02/2016 v3"

Commit message: Flipped V_AC pins
Connections:
- net V_AC+: now also B1.~2, J1.P1@2, R2.2; no longer R1.2, R2.1
- net V_AC-: now also R1.2, R2.1; no longer B1.~2, J1.P1@2, R2.2
Routing:
- net V_AC+: track 15.8 -> 35.0 mm
- net V_AC-: track 19.0 -> 7.93 mm
Other:
- board text added: "whatnick 07/03/2016 v4"
- board text removed: "whatnick 21/02/2016 v3"
Changed lines of the file:
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@@
 <?xml version="1.0" encoding="utf-8"?>
 <!DOCTYPE eagle SYSTEM "eagle.dtd">
-<eagle version="7.4.0">
+<eagle version="7.1.0">
 <drawing>
 <settings>
@@
 <layer number="17" name="Pads" color="2" fill="1" visible="yes" active="yes"/>
 <layer number="18" name="Vias" color="2" fill="1" visible="yes" active="yes"/>
-<layer number="19" name="Unrouted" color="6" fill="1" visible="no" active="yes"/>
+<layer number="19" name="Unrouted" color="6" fill="1" visible="yes" active="yes"/>
 <layer number="20" name="Dimension" color="15" fill="1" visible="yes" active="yes"/>
 <layer number="21" name="tPlace" color="7" fill="1" visible="yes" active="yes"/>
@@
 Featherwing</text>
 <text x="8.1026" y="14.2748" size="1.27" layer="22" font="vector" ratio="20" rot="MR0" align="center">whatnick
-21/02/2016 v3</text>
+07/03/2016 v4</text>
 <text x="21.0566" y="20.447" size="1.016" layer="22" font="vector" ratio="20" rot="MR180">VUSB</text>
 <text x="42.3672" y="20.7518" size="1.016" layer="22" font="vector" ratio="20" rot="MR270">SCL</text>
@@
 <attribute name="SPICEPREFIX" value="R" x="12.2936" y="20.4724" size="1.778" layer="27" rot="R180" display="off"/>
 </element>
-<element name="R2" library="resistor" package="R0603" value="10K" x="8.0264" y="20.4724" smashed="yes" rot="R180">
-<attribute name="NAME" x="7.112" y="21.2344" size="1.016" layer="25" font="vector" ratio="20"/>
-<attribute name="VALUE" x="8.6614" y="22.3774" size="1.27" layer="27" rot="R180"/>
-<attribute name="SPICEPREFIX" value="R" x="8.0264" y="20.4724" size="1.778" layer="27" rot="R180" display="off"/>
+<element name="R2" library="resistor" package="R0603" value="10K" x="8.0518" y="20.4724" smashed="yes" rot="R180">
+<attribute name="NAME" x="7.1374" y="21.2344" size="1.016" layer="25" font="vector" ratio="20"/>
+<attribute name="VALUE" x="8.6868" y="22.3774" size="1.27" layer="27" rot="R180"/>
+<attribute name="SPICEPREFIX" value="R" x="8.0518" y="20.4724" size="1.778" layer="27" rot="R180" display="off"/>
 </element>
 <element name="B1" library="rectifier" package="SOIC-4" value="MB8S" x="20.3962" y="14.6304" smashed="yes" rot="R270">
@@
 </signal>
 <signal name="V_AC+">
-<contactref element="R2" pad="1"/>
-<contactref element="R1" pad="2"/>
 <contactref element="R7" pad="1"/>
-<wire x1="11.3792" y1="20.5232" x2="8.9408" y2="20.5232" width="0.254" layer="1"/>
-<wire x1="8.9408" y1="20.5232" x2="8.8764" y2="20.4724" width="0.254" layer="1"/>
-<wire x1="11.3792" y1="20.5232" x2="11.4436" y2="20.4724" width="0.254" layer="1"/>
-<wire x1="16.764" y1="17.5768" x2="16.4592" y2="17.8816" width="0.254" layer="16"/>
-<wire x1="16.8656" y1="17.5768" x2="16.764" y2="17.5768" width="0.254" layer="16"/>
-<wire x1="17.3736" y1="17.0688" x2="16.8656" y2="17.5768" width="0.254" layer="16"/>
-<wire x1="17.5768" y1="17.0688" x2="17.3736" y2="17.0688" width="0.254" layer="1"/>
+<contactref element="B1" pad="~2"/>
+<contactref element="J1" pad="P1@2"/>
+<contactref element="R2" pad="2"/>
+<wire x1="5.3975" y1="18.7325" x2="6.985" y2="20.32" width="0.254" layer="1"/>
+<wire x1="5.3975" y1="17.145" x2="5.3975" y2="18.0975" width="0.254" layer="1"/>
+<wire x1="5.3975" y1="18.0975" x2="5.3975" y2="18.7325" width="0.254" layer="1"/>
+<wire x1="6.985" y1="20.32" x2="7.2018" y2="20.4724" width="0.254" layer="1"/>
+<wire x1="5.3975" y1="17.145" x2="5.395" y2="17.13" width="0.254" layer="1"/>
+<wire x1="12.7" y1="13.335" x2="17.145" y2="13.335" width="0.254" layer="1"/>
+<wire x1="12.7" y1="13.6525" x2="12.7" y2="13.335" width="0.254" layer="1"/>
+<wire x1="10.795" y1="15.5575" x2="12.7" y2="13.6525" width="0.254" layer="1"/>
+<wire x1="7.9375" y1="15.5575" x2="10.795" y2="15.5575" width="0.254" layer="1"/>
+<wire x1="5.3975" y1="18.0975" x2="7.9375" y2="15.5575" width="0.254" layer="1"/>
+<wire x1="17.145" y1="13.335" x2="17.3462" y2="13.3304" width="0.254" layer="1"/>
+<wire x1="5.3975" y1="18.0975" x2="5.395" y2="17.13" width="0.254" layer="1"/>
+<wire x1="17.272" y1="17.0688" x2="16.4592" y2="17.8816" width="0.254" layer="16"/>
+<wire x1="17.5768" y1="17.0688" x2="17.272" y2="17.0688" width="0.254" layer="16"/>
 <wire x1="18.0848" y1="17.5768" x2="17.5768" y2="17.0688" width="0.254" layer="1"/>
 <wire x1="18.0848" y1="18.1864" x2="18.0848" y2="17.5768" width="0.254" layer="1"/>
-<wire x1="17.78" y1="18.4912" x2="18.0848" y2="18.1864" width="0.254" layer="1"/>
-<wire x1="16.8656" y1="18.4912" x2="17.78" y2="18.4912" width="0.254" layer="1"/>
-<wire x1="16.4592" y1="18.8976" x2="16.8656" y2="18.4912" width="0.254" layer="1"/>
-<wire x1="16.4592" y1="19.304" x2="16.4592" y2="18.8976" width="0.254" layer="1"/>
-<wire x1="15.748" y1="20.0152" x2="16.4592" y2="19.304" width="0.254" layer="1"/>
-<wire x1="15.6464" y1="20.0152" x2="15.748" y2="20.0152" width="0.254" layer="1"/>
-<wire x1="15.0368" y1="20.6248" x2="15.6464" y2="20.0152" width="0.254" layer="1"/>
-<wire x1="15.0368" y1="20.9296" x2="15.0368" y2="20.6248" width="0.254" layer="1"/>
-<wire x1="13.5128" y1="22.4536" x2="15.0368" y2="20.9296" width="0.254" layer="1"/>
-<wire x1="12.3952" y1="22.4536" x2="13.5128" y2="22.4536" width="0.254" layer="1"/>
-<wire x1="11.5824" y1="21.6408" x2="12.3952" y2="22.4536" width="0.254" layer="1"/>
-<wire x1="11.5824" y1="20.828" x2="11.5824" y2="21.6408" width="0.254" layer="1"/>
-<wire x1="11.3792" y1="20.6248" x2="11.5824" y2="20.828" width="0.254" layer="1"/>
+<wire x1="17.6784" y1="18.5928" x2="18.0848" y2="18.1864" width="0.254" layer="1"/>
+<wire x1="16.764" y1="18.5928" x2="17.6784" y2="18.5928" width="0.254" layer="1"/>
+<wire x1="16.256" y1="19.1008" x2="16.764" y2="18.5928" width="0.254" layer="1"/>
+<wire x1="16.256" y1="19.7104" x2="16.256" y2="19.1008" width="0.254" layer="1"/>
+<wire x1="14.6304" y1="21.336" x2="16.256" y2="19.7104" width="0.254" layer="1"/>
+<wire x1="8.128" y1="21.336" x2="14.6304" y2="21.336" width="0.254" layer="1"/>
+<wire x1="7.3152" y1="20.5232" x2="8.128" y2="21.336" width="0.254" layer="1"/>
 <wire x1="16.4592" y1="17.8816" x2="16.4338" y2="17.9696" width="0.254" layer="16"/>
-<wire x1="11.3792" y1="20.6248" x2="11.4436" y2="20.4724" width="0.254" layer="1"/>
-<via x="17.3736" y="17.0688" extent="1-16" drill="0.3048"/>
+<wire x1="7.3152" y1="20.5232" x2="7.2018" y2="20.4724" width="0.254" layer="1"/>
+<via x="17.5768" y="17.0688" extent="1-16" drill="0.3048"/>
 </signal>
 <signal name="V_AC-" class="1">
-<contactref element="J1" pad="P1@2"/>
-<contactref element="B1" pad="~2"/>
-<contactref element="R2" pad="2"/>
 <contactref element="R9" pad="1"/>
-<wire x1="14.0208" y1="15.5448" x2="14.0208" y2="16.1544" width="0.3048" layer="16"/>
-<wire x1="14.4272" y1="15.1384" x2="14.0208" y2="15.5448" width="0.3048" layer="16"/>
-<wire x1="16.0528" y1="13.5128" x2="14.4272" y2="15.1384" width="0.3048" layer="1"/>
-<wire x1="17.1704" y1="13.5128" x2="16.0528" y2="13.5128" width="0.3048" layer="1"/>
-<wire x1="17.272" y1="13.4112" x2="17.1704" y2="13.5128" width="0.3048" layer="1"/>
-<wire x1="14.0208" y1="16.1544" x2="13.9446" y2="16.1934" width="0.3048" layer="16"/>
-<wire x1="17.272" y1="13.4112" x2="17.3462" y2="13.3304" width="0.3048" layer="1"/>
-<wire x1="7.112" y1="19.4056" x2="7.112" y2="20.4216" width="0.3048" layer="1"/>
-<wire x1="5.4864" y1="17.78" x2="7.112" y2="19.4056" width="0.3048" layer="1"/>
-<wire x1="5.4864" y1="17.1704" x2="5.4864" y2="17.78" width="0.3048" layer="1"/>
-<wire x1="7.112" y1="20.4216" x2="7.1764" y2="20.4724" width="0.3048" layer="1"/>
-<wire x1="5.4864" y1="17.1704" x2="5.395" y2="17.13" width="0.3048" layer="1"/>
-<wire x1="8.636" y1="15.0368" x2="14.3256" y2="15.0368" width="0.3048" layer="1"/>
-<wire x1="6.604" y1="17.0688" x2="8.636" y2="15.0368" width="0.3048" layer="1"/>
-<wire x1="5.588" y1="17.0688" x2="6.604" y2="17.0688" width="0.3048" layer="1"/>
-<wire x1="14.3256" y1="15.0368" x2="14.4272" y2="15.1384" width="0.3048" layer="1"/>
-<wire x1="5.588" y1="17.0688" x2="5.395" y2="17.13" width="0.3048" layer="1"/>
-<via x="14.4272" y="15.1384" extent="1-16" drill="0.3048"/>
+<contactref element="R1" pad="2"/>
+<contactref element="R2" pad="1"/>
+<wire x1="11.3792" y1="20.5232" x2="8.9408" y2="20.5232" width="0.3048" layer="1"/>
+<wire x1="8.9408" y1="20.5232" x2="8.9018" y2="20.4724" width="0.3048" layer="1"/>
+<wire x1="11.3792" y1="20.5232" x2="11.4436" y2="20.4724" width="0.3048" layer="1"/>
+<wire x1="12.5984" y1="17.5768" x2="13.9192" y2="16.256" width="0.3048" layer="16"/>
+<wire x1="12.5984" y1="19.4056" x2="12.5984" y2="17.5768" width="0.3048" layer="16"/>
+<wire x1="11.5824" y1="20.4216" x2="12.5984" y2="19.4056" width="0.3048" layer="1"/>
+<wire x1="13.9192" y1="16.256" x2="13.9446" y2="16.1934" width="0.3048" layer="16"/>
+<wire x1="11.5824" y1="20.4216" x2="11.4436" y2="20.4724" width="0.3048" layer="1"/>
+<via x="12.5984" y="19.4056" extent="1-16" drill="0.3048"/>
 </signal>
 <signal name="N$1">
