File: ADS1115_Featherwing.sch (EAGLE design)
At the start: 24 parts, among them J2 ST-PJ-312, U1 ADS1115IDGST

Commit message: Rewired fixed board
Connections:
- net N$4: now also U$7.VIN; no longer U$7.VOUT
- net REOUT: now also U$7.VOUT; no longer U$7.VIN
Changed lines of the file:
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@@
 <clearance class="0" value="0.1524"/>
 </class>
-<class number="1" name="pwr" width="0.8128" drill="0">
-<clearance class="1" value="0.254"/>
+<class number="1" name="pwr" width="0.6096" drill="0">
+<clearance class="1" value="0.1524"/>
 </class>
 </classes>
@@
 <instance part="B2" gate="G$1" x="121.92" y="114.3" rot="MR0"/>
 <instance part="J4" gate="J" x="157.48" y="114.3" rot="R180"/>
-<instance part="U$7" gate="G$1" x="106.68" y="111.76"/>
+<instance part="U$7" gate="G$1" x="66.04" y="111.76" rot="MR0"/>
 <instance part="C3" gate="G$1" x="68.58" y="114.3"/>
 <instance part="C4" gate="G$1" x="101.6" y="114.3"/>
@@
 </segment>
 </net>
-<net name="VDD" class="0">
+<net name="VDD" class="1">
 <segment>
 <pinref part="R1" gate="G$1" pin="1"/>
@@
 </segment>
 </net>
-<net name="AIN0" class="0">
+<net name="AIN0" class="1">
 <segment>
 <pinref part="U1" gate="G$1" pin="AIN0"/>
@@
 <segment>
 <label x="66.04" y="119.38" size="1.778" layer="95"/>
-<pinref part="U$7" gate="G$1" pin="VIN"/>
-<wire x1="73.66" y1="119.38" x2="68.58" y2="119.38" width="0.1524" layer="91"/>
 <wire x1="68.58" y1="119.38" x2="67.31" y2="119.38" width="0.1524" layer="91"/>
 <wire x1="68.58" y1="119.38" x2="68.58" y2="116.84" width="0.1524" layer="91"/>
-<junction x="68.58" y="119.38"/>
 <pinref part="C3" gate="G$1" pin="1"/>
 <pinref part="D2" gate="G$1" pin="+"/>
+<pinref part="U$7" gate="G$1" pin="VOUT"/>
+<wire x1="73.66" y1="119.38" x2="68.58" y2="119.38" width="0.1524" layer="91"/>
+<junction x="68.58" y="119.38"/>
 </segment>
 </net>
@@
 <wire x1="109.22" y1="119.38" x2="101.6" y2="119.38" width="0.1524" layer="91"/>
 <wire x1="101.6" y1="119.38" x2="101.6" y2="116.84" width="0.1524" layer="91"/>
+<pinref part="B2" gate="G$1" pin="+"/>
+<wire x1="109.22" y1="114.3" x2="116.84" y2="114.3" width="0.1524" layer="91"/>
+<pinref part="C4" gate="G$1" pin="1"/>
+<pinref part="U$7" gate="G$1" pin="VIN"/>
 <wire x1="101.6" y1="119.38" x2="99.06" y2="119.38" width="0.1524" layer="91"/>
 <junction x="101.6" y="119.38"/>
-<pinref part="B2" gate="G$1" pin="+"/>
-<wire x1="109.22" y1="114.3" x2="116.84" y2="114.3" width="0.1524" layer="91"/>
-<pinref part="U$7" gate="G$1" pin="VOUT"/>
-<pinref part="C4" gate="G$1" pin="1"/>
-</segment>
-</net>
-<net name="USB" class="0">
+</segment>
+</net>
+<net name="USB" class="1">
 <segment>
 <label x="55.88" y="119.38" size="1.778" layer="95" rot="R180" xref="yes"/>

Commit message: Added grove connector
Parts:
- added J1: 4P-SMD-2.0-90D, Seeed-OPL-Connector:GROVE-CONNECTOR-SMD-90D(4+2P-2.0)
Connections:
- removed net N$1: C2.P$1, FB1.P$1
- removed net N$2: C2.P$2, FB2.P$1
- new net 3V: C2.P$1, FB1.P$1, J1.3, MS1.3V
- new net AGND: B2.-, C2.P$2, C3.2, C4.2, FB2.P$1, J1.4, MS1.GND, U$7.GND
- net GND: now also J1.SS1, J1.SS2; no longer B2.-, C3.2, C4.2, U$7.GND
- net SCL: now also J1.1
- net SDA: now also J1.2
- net VDD: no longer MS1.3V
Changed lines of the file:
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@@
 <clearance class="0" value="0.1524"/>
 </class>
-<class number="1" name="pwr" width="0.6096" drill="0">
+<class number="1" name="pwr" width="0.3048" drill="0">
 <clearance class="1" value="0.1524"/>
 </class>
@@
 <part name="R6" library="resistor" deviceset="R-EU_" device="R0603" value="100K"/>
 <part name="R7" library="resistor" deviceset="R-EU_" device="R0603" value="10K"/>
-<part name="U$1" library="Power or GND " deviceset="GND_POWER" device=""/>
 <part name="B2" library="rectifier" deviceset="MB*S" device="" technology="8"/>
 <part name="J4" library="dp_devices" deviceset="CON_DC_M" device="-DC_SMD"/>
@@
 <part name="C4" library="adafruit" deviceset="C-US" device="C1206" value="10uF"/>
 <part name="D2" library="Seeed-OPL-Diode" deviceset="SMD-DIODE-SCHOTTKY-20V-1A(SOD-123)" device="" value="20V-1A"/>
+<part name="J1" library="Seeed-OPL-Connector" deviceset="GROVE-CONNECTOR-SMD-90D(4+2P-2.0)" device="" value="4P-SMD-2.0-90D"/>
 </parts>
 <sheets>
@@
 <instance part="R6" gate="G$1" x="139.7" y="121.92" rot="R270"/>
 <instance part="R7" gate="G$1" x="139.7" y="106.68" rot="R270"/>
-<instance part="U$1" gate="G$1" x="90.17" y="104.14"/>
 <instance part="B2" gate="G$1" x="121.92" y="114.3" rot="MR0"/>
 <instance part="J4" gate="J" x="157.48" y="114.3" rot="R180"/>
@@
 <instance part="C4" gate="G$1" x="101.6" y="114.3"/>
 <instance part="D2" gate="G$1" x="63.5" y="119.38" rot="R180"/>
+<instance part="J1" gate="G$1" x="-12.7" y="7.62"/>
 </instances>
 <busses>
 </busses>
 <nets>
-<net name="GND" class="0">
+<net name="GND" class="1">
 <segment>
 <pinref part="C1" gate="G$1" pin="P$1"/>
@@
 </segment>
 <segment>
-<wire x1="68.58" y1="109.22" x2="68.58" y2="104.14" width="0.1524" layer="91"/>
-<wire x1="68.58" y1="104.14" x2="86.36" y2="104.14" width="0.1524" layer="91"/>
-<wire x1="101.6" y1="104.14" x2="101.6" y2="109.22" width="0.1524" layer="91"/>
-<wire x1="86.36" y1="104.14" x2="90.17" y2="104.14" width="0.1524" layer="91"/>
-<junction x="86.36" y="104.14"/>
-<wire x1="90.17" y1="104.14" x2="101.6" y2="104.14" width="0.1524" layer="91"/>
-<pinref part="U$1" gate="G$1" pin="GND"/>
-<junction x="90.17" y="104.14"/>
-<pinref part="U$7" gate="G$1" pin="GND"/>
-<junction x="86.36" y="104.14"/>
-<pinref part="C3" gate="G$1" pin="2"/>
-<pinref part="C4" gate="G$1" pin="2"/>
-<junction x="101.6" y="104.14"/>
-<pinref part="B2" gate="G$1" pin="-"/>
-<wire x1="127" y1="114.3" x2="129.54" y2="114.3" width="0.1524" layer="91"/>
-<wire x1="129.54" y1="114.3" x2="129.54" y2="104.14" width="0.1524" layer="91"/>
-<wire x1="101.6" y1="104.14" x2="129.54" y2="104.14" width="0.1524" layer="91"/>
+<pinref part="J1" gate="G$1" pin="SS1"/>
+<wire x1="-12.7" y1="15.24" x2="-7.62" y2="15.24" width="0.1524" layer="91"/>
+<wire x1="-7.62" y1="15.24" x2="-7.62" y2="0" width="0.1524" layer="91"/>
+<pinref part="J1" gate="G$1" pin="SS2"/>
+<wire x1="-7.62" y1="0" x2="-12.7" y2="0" width="0.1524" layer="91"/>
+<label x="-7.62" y="7.62" size="1.778" layer="95" xref="yes"/>
 </segment>
 </net>
@@
 <label x="-40.64" y="78.74" size="1.778" layer="95" rot="R90"/>
 </segment>
+<segment>
+<pinref part="J1" gate="G$1" pin="1"/>
+<wire x1="-17.78" y1="11.43" x2="-24.638" y2="11.43" width="0.1524" layer="91"/>
+<label x="-24.892" y="11.43" size="1.778" layer="95" rot="R180" xref="yes"/>
+</segment>
 </net>
 <net name="SDA" class="0">
@@
 <wire x1="-43.18" y1="83.82" x2="-43.18" y2="76.2" width="0.1524" layer="91"/>
 <label x="-43.18" y="78.74" size="1.778" layer="95" rot="R90"/>
+</segment>
+<segment>
+<label x="-23.876" y="8.89" size="1.778" layer="95" rot="R180" xref="yes"/>
+<pinref part="J1" gate="G$1" pin="2"/>
+<wire x1="-17.78" y1="8.89" x2="-23.876" y2="8.89" width="0.1524" layer="91"/>
 </segment>
 </net>
@@
 <label x="50.8" y="7.62" size="1.778" layer="95" rot="R90"/>
 </segment>
-<segment>
-<pinref part="MS1" gate="G$1" pin="3V"/>
-<wire x1="-7.62" y1="127" x2="-7.62" y2="137.16" width="0.1524" layer="91"/>
-<label x="-5.08" y="129.54" size="1.778" layer="95" rot="R90"/>
-</segment>
 </net>
 <net name="ALERT" class="0">
@@
 </segment>
 </net>
-<net name="N$2" class="0">
+<net name="AGND" class="1">
 <segment>
 <pinref part="FB2" gate="G$1" pin="P$1"/>
@@
 <wire x1="-27.94" y1="53.34" x2="-27.94" y2="50.8" width="0.1524" layer="91"/>
 <junction x="-27.94" y="50.8"/>
-</segment>
-</net>
-<net name="N$1" class="0">
-<segment>
-<pinref part="FB1" gate="G$1" pin="P$1"/>
-<wire x1="-22.86" y1="63.5" x2="-27.94" y2="63.5" width="0.1524" layer="91"/>
-<wire x1="-27.94" y1="63.5" x2="-35.56" y2="63.5" width="0.1524" layer="91"/>
-<wire x1="-35.56" y1="63.5" x2="-35.56" y2="53.34" width="0.1524" layer="91"/>
-<wire x1="-35.56" y1="53.34" x2="-43.18" y2="53.34" width="0.1524" layer="91"/>
-<pinref part="C2" gate="G$1" pin="P$1"/>
-<wire x1="-27.94" y1="63.5" x2="-27.94" y2="60.96" width="0.1524" layer="91"/>
-<junction x="-27.94" y="63.5"/>
+<label x="-40.64" y="50.8" size="1.778" layer="95"/>
+</segment>
+<segment>
+<pinref part="MS1" gate="G$1" pin="GND"/>
+<wire x1="-12.7" y1="127" x2="-12.7" y2="137.16" width="0.1524" layer="91"/>
+<label x="-12.7" y="129.54" size="1.778" layer="95" rot="R90"/>
+</segment>
+<segment>
+<pinref part="J1" gate="G$1" pin="4"/>
+<wire x1="-17.78" y1="3.81" x2="-24.13" y2="3.81" width="0.1524" layer="91"/>
+<label x="-24.13" y="3.81" size="1.778" layer="95" rot="R180" xref="yes"/>
+</segment>
+<segment>
+<wire x1="68.58" y1="109.22" x2="68.58" y2="104.14" width="0.1524" layer="91"/>
+<wire x1="68.58" y1="104.14" x2="86.36" y2="104.14" width="0.1524" layer="91"/>
+<wire x1="101.6" y1="104.14" x2="101.6" y2="109.22" width="0.1524" layer="91"/>
+<junction x="86.36" y="104.14"/>
+<wire x1="86.36" y1="104.14" x2="101.6" y2="104.14" width="0.1524" layer="91"/>
+<pinref part="U$7" gate="G$1" pin="GND"/>
+<junction x="86.36" y="104.14"/>
+<pinref part="C3" gate="G$1" pin="2"/>
+<pinref part="C4" gate="G$1" pin="2"/>
+<junction x="101.6" y="104.14"/>
+<pinref part="B2" gate="G$1" pin="-"/>
+<wire x1="127" y1="114.3" x2="129.54" y2="114.3" width="0.1524" layer="91"/>
+<wire x1="129.54" y1="114.3" x2="129.54" y2="104.14" width="0.1524" layer="91"/>
+<wire x1="101.6" y1="104.14" x2="129.54" y2="104.14" width="0.1524" layer="91"/>
+<label x="96.52" y="104.14" size="1.778" layer="95" rot="R270" xref="yes"/>
 </segment>
 </net>
@@
 </segment>
 </net>
+<net name="3V" class="1">
+<segment>
+<pinref part="MS1" gate="G$1" pin="3V"/>
+<wire x1="-7.62" y1="127" x2="-7.62" y2="137.16" width="0.1524" layer="91"/>
+<label x="-5.08" y="129.54" size="1.778" layer="95" rot="R90"/>
+</segment>
+<segment>
+<pinref part="FB1" gate="G$1" pin="P$1"/>
+<wire x1="-22.86" y1="63.5" x2="-27.94" y2="63.5" width="0.1524" layer="91"/>
+<wire x1="-27.94" y1="63.5" x2="-35.56" y2="63.5" width="0.1524" layer="91"/>
+<wire x1="-35.56" y1="63.5" x2="-35.56" y2="53.34" width="0.1524" layer="91"/>
+<wire x1="-35.56" y1="53.34" x2="-43.18" y2="53.34" width="0.1524" layer="91"/>
+<pinref part="C2" gate="G$1" pin="P$1"/>
+<wire x1="-27.94" y1="63.5" x2="-27.94" y2="60.96" width="0.1524" layer="91"/>
+<junction x="-27.94" y="63.5"/>
+<label x="-40.64" y="53.34" size="1.778" layer="95"/>
+</segment>
+<segment>
+<label x="-24.13" y="6.35" size="1.778" layer="95" rot="R180" xref="yes"/>
+<pinref part="J1" gate="G$1" pin="3"/>
+<wire x1="-17.78" y1="6.35" x2="-23.876" y2="6.35" width="0.1524" layer="91"/>
+</segment>
+</net>

Commit message: Switched to 50V electrolytic
Parts:
- removed C3: 100uF, adafruit:C-USC1210
- added C5: 100uF 50V, adafruit:CPOL-US153CLV-0810
- C4: value 10uF -> 10uF 50V
Connections:
- net AGND: now also C5.-; no longer C3.2
- net N$4: now also C5.+; no longer C4.1
- net REOUT: now also C4.1; no longer C3.1
Other:
- moved on the sheet: C4
Changed lines of the file:
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@@
 <?xml version="1.0" encoding="utf-8"?>
 <!DOCTYPE eagle SYSTEM "eagle.dtd">
-<eagle version="7.4.0">
+<eagle version="7.1.0">
 <drawing>
 <settings>
@@
 <grid distance="0.1" unitdist="inch" unit="inch" style="lines" multiple="1" display="no" altdistance="0.01" altunitdist="inch" altunit="inch"/>
 <layers>
-<layer number="1" name="Top" color="4" fill="1" visible="no" active="no"/>
-<layer number="16" name="Bottom" color="1" fill="1" visible="no" active="no"/>
-<layer number="17" name="Pads" color="2" fill="1" visible="no" active="no"/>
-<layer number="18" name="Vias" color="2" fill="1" visible="no" active="no"/>
-<layer number="19" name="Unrouted" color="6" fill="1" visible="no" active="no"/>
-<layer number="20" name="Dimension" color="15" fill="1" visible="no" active="no"/>
-<layer number="21" name="tPlace" color="7" fill="1" visible="no" active="no"/>
-<layer number="22" name="bPlace" color="7" fill="1" visible="no" active="no"/>
-<layer number="23" name="tOrigins" color="15" fill="1" visible="no" active="no"/>
-<layer number="24" name="bOrigins" color="15" fill="1" visible="no" active="no"/>
-<layer number="25" name="tNames" color="7" fill="1" visible="no" active="no"/>
-<layer number="26" name="bNames" color="7" fill="1" visible="no" active="no"/>
-<layer number="27" name="tValues" color="7" fill="1" visible="no" active="no"/>
-<layer number="28" name="bValues" color="7" fill="1" visible="no" active="no"/>
+<layer number="1" name="Top" color="4" fill="1" visible="yes" active="no"/>
+<layer number="16" name="Bottom" color="1" fill="1" visible="yes" active="no"/>
+<layer number="17" name="Pads" color="2" fill="1" visible="yes" active="no"/>
+<layer number="18" name="Vias" color="2" fill="1" visible="yes" active="no"/>
+<layer number="19" name="Unrouted" color="6" fill="1" visible="yes" active="no"/>
+<layer number="20" name="Dimension" color="15" fill="1" visible="yes" active="no"/>
+<layer number="21" name="tPlace" color="7" fill="1" visible="yes" active="no"/>
+<layer number="22" name="bPlace" color="11" fill="1" visible="yes" active="no"/>
+<layer number="23" name="tOrigins" color="15" fill="1" visible="yes" active="no"/>
+<layer number="24" name="bOrigins" color="15" fill="1" visible="yes" active="no"/>
+<layer number="25" name="tNames" color="7" fill="1" visible="yes" active="no"/>
+<layer number="26" name="bNames" color="11" fill="1" visible="yes" active="no"/>
+<layer number="27" name="tValues" color="7" fill="1" visible="yes" active="no"/>
+<layer number="28" name="bValues" color="7" fill="1" visible="yes" active="no"/>
 <layer number="29" name="tStop" color="7" fill="3" visible="no" active="no"/>
 <layer number="30" name="bStop" color="7" fill="6" visible="no" active="no"/>
@@
 <layer number="35" name="tGlue" color="7" fill="4" visible="no" active="no"/>
 <layer number="36" name="bGlue" color="7" fill="5" visible="no" active="no"/>
-<layer number="37" name="tTest" color="7" fill="1" visible="no" active="no"/>
-<layer number="38" name="bTest" color="7" fill="1" visible="no" active="no"/>
+<layer number="37" name="tTest" color="7" fill="1" visible="yes" active="no"/>
+<layer number="38" name="bTest" color="7" fill="1" visible="yes" active="no"/>
 <layer number="39" name="tKeepout" color="4" fill="11" visible="no" active="no"/>
 <layer number="40" name="bKeepout" color="1" fill="11" visible="no" active="no"/>
@@
 <layer number="44" name="Drills" color="7" fill="1" visible="no" active="no"/>
 <layer number="45" name="Holes" color="7" fill="1" visible="no" active="no"/>
-<layer number="46" name="Milling" color="3" fill="1" visible="no" active="no"/>
-<layer number="47" name="Measures" color="7" fill="1" visible="no" active="no"/>
-<layer number="48" name="Document" color="7" fill="1" visible="no" active="no"/>
-<layer number="49" name="Reference" color="7" fill="1" visible="no" active="no"/>
-<layer number="50" name="dxf" color="7" fill="1" visible="no" active="no"/>
-<layer number="51" name="tDocu" color="7" fill="1" visible="no" active="no"/>
-<layer number="52" name="bDocu" color="7" fill="1" visible="no" active="no"/>
-<layer number="53" name="tGND_GNDA" color="7" fill="9" visible="no" active="no"/>
-<layer number="54" name="bGND_GNDA" color="1" fill="9" visible="no" active="no"/>
-<layer number="56" name="wert" color="7" fill="1" visible="no" active="no"/>
-<layer number="57" name="tCAD" color="7" fill="1" visible="no" active="no"/>
-<layer number="59" name="tCarbon" color="7" fill="1" visible="no" active="no"/>
-<layer number="60" name="bCarbon" color="7" fill="1" visible="no" active="no"/>
+<layer number="46" name="Milling" color="3" fill="1" visible="yes" active="no"/>
+<layer number="47" name="Measures" color="7" fill="1" visible="yes" active="no"/>
+<layer number="48" name="Document" color="7" fill="1" visible="yes" active="no"/>
+<layer number="49" name="Reference" color="7" fill="1" visible="yes" active="no"/>
+<layer number="50" name="dxf" color="7" fill="1" visible="yes" active="no"/>
+<layer number="51" name="tDocu" color="7" fill="1" visible="yes" active="no"/>
+<layer number="52" name="bDocu" color="7" fill="1" visible="yes" active="no"/>
+<layer number="53" name="tGND_GNDA" color="7" fill="9" visible="yes" active="no"/>
+<layer number="54" name="bGND_GNDA" color="1" fill="9" visible="yes" active="no"/>
+<layer number="56" name="wert" color="7" fill="1" visible="yes" active="no"/>
+<layer number="57" name="tCAD" color="7" fill="1" visible="yes" active="no"/>
+<layer number="59" name="tCarbon" color="7" fill="1" visible="yes" active="no"/>
+<layer number="60" name="bCarbon" color="7" fill="1" visible="yes" active="no"/>
 <layer number="90" name="Modules" color="5" fill="1" visible="yes" active="yes"/>
 <layer number="91" name="Nets" color="2" fill="1" visible="yes" active="yes"/>
@@
 <part name="J4" library="dp_devices" deviceset="CON_DC_M" device="-DC_SMD"/>
 <part name="U$7" library="recom-intl" deviceset="ROF-78E" device=""/>
-<part name="C3" library="adafruit" deviceset="C-US" device="C1210" value="100uF"/>
-<part name="C4" library="adafruit" deviceset="C-US" device="C1206" value="10uF"/>
+<part name="C4" library="adafruit" deviceset="C-US" device="C1206" value="10uF 50V"/>
 <part name="D2" library="Seeed-OPL-Diode" deviceset="SMD-DIODE-SCHOTTKY-20V-1A(SOD-123)" device="" value="20V-1A"/>
 <part name="J1" library="Seeed-OPL-Connector" deviceset="GROVE-CONNECTOR-SMD-90D(4+2P-2.0)" device="" value="4P-SMD-2.0-90D"/>
+<part name="C5" library="adafruit" deviceset="CPOL-US" device="153CLV-0810" value="100uF 50V"/>
 </parts>
 <sheets>
@@
 <instance part="J4" gate="J" x="157.48" y="114.3" rot="R180"/>
 <instance part="U$7" gate="G$1" x="66.04" y="111.76" rot="MR0"/>
-<instance part="C3" gate="G$1" x="68.58" y="114.3"/>
-<instance part="C4" gate="G$1" x="101.6" y="114.3"/>
+<instance part="C4" gate="G$1" x="68.58" y="114.3"/>
 <instance part="D2" gate="G$1" x="63.5" y="119.38" rot="R180"/>
 <instance part="J1" gate="G$1" x="-12.7" y="7.62"/>
+<instance part="C5" gate="G$1" x="101.6" y="114.3"/>
 </instances>
 <busses>
@@
 </segment>
 <segment>
-<wire x1="68.58" y1="109.22" x2="68.58" y2="104.14" width="0.1524" layer="91"/>
 <wire x1="68.58" y1="104.14" x2="86.36" y2="104.14" width="0.1524" layer="91"/>
-<wire x1="101.6" y1="104.14" x2="101.6" y2="109.22" width="0.1524" layer="91"/>
 <junction x="86.36" y="104.14"/>
 <wire x1="86.36" y1="104.14" x2="101.6" y2="104.14" width="0.1524" layer="91"/>
 <pinref part="U$7" gate="G$1" pin="GND"/>
 <junction x="86.36" y="104.14"/>
-<pinref part="C3" gate="G$1" pin="2"/>
-<pinref part="C4" gate="G$1" pin="2"/>
 <junction x="101.6" y="104.14"/>
 <pinref part="B2" gate="G$1" pin="-"/>
@@
 <wire x1="101.6" y1="104.14" x2="129.54" y2="104.14" width="0.1524" layer="91"/>
 <label x="96.52" y="104.14" size="1.778" layer="95" rot="R270" xref="yes"/>
+<pinref part="C4" gate="G$1" pin="2"/>
+<wire x1="68.58" y1="109.22" x2="68.58" y2="104.14" width="0.1524" layer="91"/>
+<pinref part="C5" gate="G$1" pin="-"/>
+<wire x1="101.6" y1="109.22" x2="101.6" y2="104.14" width="0.1524" layer="91"/>
 </segment>
 </net>
@@
 <label x="66.04" y="119.38" size="1.778" layer="95"/>
 <wire x1="68.58" y1="119.38" x2="67.31" y2="119.38" width="0.1524" layer="91"/>
-<wire x1="68.58" y1="119.38" x2="68.58" y2="116.84" width="0.1524" layer="91"/>
-<pinref part="C3" gate="G$1" pin="1"/>
 <pinref part="D2" gate="G$1" pin="+"/>
 <pinref part="U$7" gate="G$1" pin="VOUT"/>
 <wire x1="73.66" y1="119.38" x2="68.58" y2="119.38" width="0.1524" layer="91"/>
 <junction x="68.58" y="119.38"/>
+<pinref part="C4" gate="G$1" pin="1"/>
+<wire x1="68.58" y1="116.84" x2="68.58" y2="119.38" width="0.1524" layer="91"/>
 </segment>
 </net>
@@
 <wire x1="109.22" y1="114.3" x2="109.22" y2="119.38" width="0.1524" layer="91"/>
 <wire x1="109.22" y1="119.38" x2="101.6" y2="119.38" width="0.1524" layer="91"/>
-<wire x1="101.6" y1="119.38" x2="101.6" y2="116.84" width="0.1524" layer="91"/>
 <pinref part="B2" gate="G$1" pin="+"/>
 <wire x1="109.22" y1="114.3" x2="116.84" y2="114.3" width="0.1524" layer="91"/>
-<pinref part="C4" gate="G$1" pin="1"/>
 <pinref part="U$7" gate="G$1" pin="VIN"/>
 <wire x1="101.6" y1="119.38" x2="99.06" y2="119.38" width="0.1524" layer="91"/>
 <junction x="101.6" y="119.38"/>
-</segment>
-</net>
+<pinref part="C5" gate="G$1" pin="+"/>
+<wire x1="101.6" y1="116.84" x2="101.6" y2="119.38" width="0.1524" layer="91"/>
+</segment>
+</net>
