File: ADS1115_Featherwing.sch (EAGLE design)
At the start: 25 parts, among them J1 4P-SMD-2.0-90D, J2 ST-PJ-312, U1 ADS1115IDGST

Commit message: Added protection resistor
Parts:
- added R8: 10K, resistor:R-EU_R0603
Connections:
- new net N$1: R8.2, U1.AIN1
- net AIN1: now also R8.1; no longer U1.AIN1
Changed lines of the file:
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@@
 <?xml version="1.0" encoding="utf-8"?>
 <!DOCTYPE eagle SYSTEM "eagle.dtd">
-<eagle version="7.1.0">
+<eagle version="7.4.0">
 <drawing>
 <settings>
@@
 <grid distance="0.1" unitdist="inch" unit="inch" style="lines" multiple="1" display="no" altdistance="0.01" altunitdist="inch" altunit="inch"/>
 <layers>
-<layer number="1" name="Top" color="4" fill="1" visible="yes" active="no"/>
-<layer number="16" name="Bottom" color="1" fill="1" visible="yes" active="no"/>
-<layer number="17" name="Pads" color="2" fill="1" visible="yes" active="no"/>
-<layer number="18" name="Vias" color="2" fill="1" visible="yes" active="no"/>
-<layer number="19" name="Unrouted" color="6" fill="1" visible="yes" active="no"/>
-<layer number="20" name="Dimension" color="15" fill="1" visible="yes" active="no"/>
-<layer number="21" name="tPlace" color="7" fill="1" visible="yes" active="no"/>
-<layer number="22" name="bPlace" color="11" fill="1" visible="yes" active="no"/>
-<layer number="23" name="tOrigins" color="15" fill="1" visible="yes" active="no"/>
-<layer number="24" name="bOrigins" color="15" fill="1" visible="yes" active="no"/>
-<layer number="25" name="tNames" color="7" fill="1" visible="yes" active="no"/>
-<layer number="26" name="bNames" color="11" fill="1" visible="yes" active="no"/>
-<layer number="27" name="tValues" color="7" fill="1" visible="yes" active="no"/>
-<layer number="28" name="bValues" color="7" fill="1" visible="yes" active="no"/>
+<layer number="1" name="Top" color="4" fill="1" visible="no" active="no"/>
+<layer number="16" name="Bottom" color="1" fill="1" visible="no" active="no"/>
+<layer number="17" name="Pads" color="2" fill="1" visible="no" active="no"/>
+<layer number="18" name="Vias" color="2" fill="1" visible="no" active="no"/>
+<layer number="19" name="Unrouted" color="6" fill="1" visible="no" active="no"/>
+<layer number="20" name="Dimension" color="15" fill="1" visible="no" active="no"/>
+<layer number="21" name="tPlace" color="7" fill="1" visible="no" active="no"/>
+<layer number="22" name="bPlace" color="11" fill="1" visible="no" active="no"/>
+<layer number="23" name="tOrigins" color="15" fill="1" visible="no" active="no"/>
+<layer number="24" name="bOrigins" color="15" fill="1" visible="no" active="no"/>
+<layer number="25" name="tNames" color="7" fill="1" visible="no" active="no"/>
+<layer number="26" name="bNames" color="11" fill="1" visible="no" active="no"/>
+<layer number="27" name="tValues" color="7" fill="1" visible="no" active="no"/>
+<layer number="28" name="bValues" color="7" fill="1" visible="no" active="no"/>
 <layer number="29" name="tStop" color="7" fill="3" visible="no" active="no"/>
 <layer number="30" name="bStop" color="7" fill="6" visible="no" active="no"/>
@@
 <layer number="35" name="tGlue" color="7" fill="4" visible="no" active="no"/>
 <layer number="36" name="bGlue" color="7" fill="5" visible="no" active="no"/>
-<layer number="37" name="tTest" color="7" fill="1" visible="yes" active="no"/>
-<layer number="38" name="bTest" color="7" fill="1" visible="yes" active="no"/>
+<layer number="37" name="tTest" color="7" fill="1" visible="no" active="no"/>
+<layer number="38" name="bTest" color="7" fill="1" visible="no" active="no"/>
 <layer number="39" name="tKeepout" color="4" fill="11" visible="no" active="no"/>
 <layer number="40" name="bKeepout" color="1" fill="11" visible="no" active="no"/>
@@
 <layer number="44" name="Drills" color="7" fill="1" visible="no" active="no"/>
 <layer number="45" name="Holes" color="7" fill="1" visible="no" active="no"/>
-<layer number="46" name="Milling" color="3" fill="1" visible="yes" active="no"/>
-<layer number="47" name="Measures" color="7" fill="1" visible="yes" active="no"/>
-<layer number="48" name="Document" color="7" fill="1" visible="yes" active="no"/>
-<layer number="49" name="Reference" color="7" fill="1" visible="yes" active="no"/>
-<layer number="50" name="dxf" color="7" fill="1" visible="yes" active="no"/>
-<layer number="51" name="tDocu" color="7" fill="1" visible="yes" active="no"/>
-<layer number="52" name="bDocu" color="7" fill="1" visible="yes" active="no"/>
-<layer number="53" name="tGND_GNDA" color="7" fill="9" visible="yes" active="no"/>
-<layer number="54" name="bGND_GNDA" color="1" fill="9" visible="yes" active="no"/>
-<layer number="56" name="wert" color="7" fill="1" visible="yes" active="no"/>
-<layer number="57" name="tCAD" color="7" fill="1" visible="yes" active="no"/>
-<layer number="59" name="tCarbon" color="7" fill="1" visible="yes" active="no"/>
-<layer number="60" name="bCarbon" color="7" fill="1" visible="yes" active="no"/>
+<layer number="46" name="Milling" color="3" fill="1" visible="no" active="no"/>
+<layer number="47" name="Measures" color="7" fill="1" visible="no" active="no"/>
+<layer number="48" name="Document" color="7" fill="1" visible="no" active="no"/>
+<layer number="49" name="Reference" color="7" fill="1" visible="no" active="no"/>
+<layer number="50" name="dxf" color="7" fill="1" visible="no" active="no"/>
+<layer number="51" name="tDocu" color="7" fill="1" visible="no" active="no"/>
+<layer number="52" name="bDocu" color="7" fill="1" visible="no" active="no"/>
+<layer number="53" name="tGND_GNDA" color="7" fill="9" visible="no" active="no"/>
+<layer number="54" name="bGND_GNDA" color="1" fill="9" visible="no" active="no"/>
+<layer number="56" name="wert" color="7" fill="1" visible="no" active="no"/>
+<layer number="57" name="tCAD" color="7" fill="1" visible="no" active="no"/>
+<layer number="59" name="tCarbon" color="7" fill="1" visible="no" active="no"/>
+<layer number="60" name="bCarbon" color="7" fill="1" visible="no" active="no"/>
 <layer number="90" name="Modules" color="5" fill="1" visible="yes" active="yes"/>
 <layer number="91" name="Nets" color="2" fill="1" visible="yes" active="yes"/>
@@
 <part name="J1" library="Seeed-OPL-Connector" deviceset="GROVE-CONNECTOR-SMD-90D(4+2P-2.0)" device="" value="4P-SMD-2.0-90D"/>
 <part name="C5" library="adafruit" deviceset="CPOL-US" device="153CLV-0810" value="100uF 50V"/>
+<part name="R8" library="resistor" deviceset="R-EU_" device="R0603" value="10K"/>
 </parts>
 <sheets>
@@
 <instance part="J1" gate="G$1" x="-12.7" y="7.62"/>
 <instance part="C5" gate="G$1" x="101.6" y="114.3"/>
+<instance part="R8" gate="G$1" x="27.94" y="43.18"/>
 </instances>
 <busses>
@@
 <net name="AIN0" class="1">
 <segment>
+<label x="15.24" y="45.72" size="1.778" layer="95"/>
+<wire x1="15.24" y1="45.72" x2="35.56" y2="45.72" width="0.1524" layer="91"/>
 <pinref part="U1" gate="G$1" pin="AIN0"/>
-<wire x1="35.56" y1="45.72" x2="25.4" y2="45.72" width="0.1524" layer="91"/>
-<label x="15.24" y="45.72" size="1.778" layer="95"/>
-<wire x1="25.4" y1="45.72" x2="15.24" y2="45.72" width="0.1524" layer="91"/>
 </segment>
 <segment>
@@
 <net name="AIN1" class="0">
 <segment>
-<pinref part="U1" gate="G$1" pin="AIN1"/>
-<wire x1="35.56" y1="43.18" x2="15.24" y2="43.18" width="0.1524" layer="91"/>
-<label x="15.24" y="43.18" size="1.778" layer="95"/>
-</segment>
-<segment>
 <wire x1="-43.18" y1="35.56" x2="-27.94" y2="35.56" width="0.1524" layer="91"/>
 <label x="-38.1" y="35.56" size="1.778" layer="95"/>
@@
 <junction x="139.7" y="114.3"/>
 <label x="132.08" y="114.3" size="1.778" layer="95"/>
+</segment>
+<segment>
+<pinref part="R8" gate="G$1" pin="1"/>
+<wire x1="22.86" y1="43.18" x2="15.24" y2="43.18" width="0.1524" layer="91"/>
+<label x="15.24" y="43.18" size="1.778" layer="95"/>
 </segment>
 </net>
@@
 </segment>
 </net>
+<net name="N$1" class="0">
+<segment>
+<pinref part="U1" gate="G$1" pin="AIN1"/>
+<pinref part="R8" gate="G$1" pin="2"/>
+<wire x1="35.56" y1="43.18" x2="33.02" y2="43.18" width="0.1524" layer="91"/>
+</segment>
+</net>

Commit message: Switched to XP Power Vreg
Parts:
- removed U$7: ROF-78E, recom-intl:ROF-78E
- added U2: SR05, Seeed-OPL-ic:PMIC-L7805CV-DG(TO-220)ALT
- C4: value 10uF 50V -> 10uF; device adafruit:C-USC1206 -> adafruit:CPOL-US153CLV-0405
- renumbered C5 to C3
Connections:
- removed net REOUT: C4.1, D2.+, U$7.VOUT
- new net N$2: C4.+, D2.+, U2.OUT
- net AGND: now also C4.-, U2.GND; no longer C4.2, U$7.GND
- net N$4: now also U2.IN; no longer U$7.VIN
Other:
- moved on the sheet: D2
Changed lines of the file:
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@@
 <?xml version="1.0" encoding="utf-8"?>
 <!DOCTYPE eagle SYSTEM "eagle.dtd">
-<eagle version="7.4.0">
+<eagle version="7.1.0">
 <drawing>
 <settings>
@@
 <part name="B2" library="rectifier" deviceset="MB*S" device="" technology="8"/>
 <part name="J4" library="dp_devices" deviceset="CON_DC_M" device="-DC_SMD"/>
-<part name="U$7" library="recom-intl" deviceset="ROF-78E" device=""/>
-<part name="C4" library="adafruit" deviceset="C-US" device="C1206" value="10uF 50V"/>
 <part name="D2" library="Seeed-OPL-Diode" deviceset="SMD-DIODE-SCHOTTKY-20V-1A(SOD-123)" device="" value="20V-1A"/>
 <part name="J1" library="Seeed-OPL-Connector" deviceset="GROVE-CONNECTOR-SMD-90D(4+2P-2.0)" device="" value="4P-SMD-2.0-90D"/>
-<part name="C5" library="adafruit" deviceset="CPOL-US" device="153CLV-0810" value="100uF 50V"/>
+<part name="C3" library="adafruit" deviceset="CPOL-US" device="153CLV-0810" value="100uF 50V"/>
 <part name="R8" library="resistor" deviceset="R-EU_" device="R0603" value="10K"/>
+<part name="C4" library="adafruit" deviceset="CPOL-US" device="153CLV-0405" value="10uF"/>
+<part name="U2" library="Seeed-OPL-ic" deviceset="PMIC-L7805CV-DG(TO-220)" device="ALT" value="SR05"/>
 </parts>
 <sheets>
@@
 <instance part="B2" gate="G$1" x="121.92" y="114.3" rot="MR0"/>
 <instance part="J4" gate="J" x="157.48" y="114.3" rot="R180"/>
-<instance part="U$7" gate="G$1" x="66.04" y="111.76" rot="MR0"/>
-<instance part="C4" gate="G$1" x="68.58" y="114.3"/>
-<instance part="D2" gate="G$1" x="63.5" y="119.38" rot="R180"/>
+<instance part="D2" gate="G$1" x="60.96" y="119.38" rot="R180"/>
 <instance part="J1" gate="G$1" x="-12.7" y="7.62"/>
-<instance part="C5" gate="G$1" x="101.6" y="114.3"/>
+<instance part="C3" gate="G$1" x="101.6" y="114.3"/>
 <instance part="R8" gate="G$1" x="27.94" y="43.18"/>
+<instance part="C4" gate="G$1" x="66.04" y="114.3"/>
+<instance part="U2" gate="G$1" x="83.82" y="119.38" rot="MR0"/>
 </instances>
 <busses>
@@
 </segment>
 <segment>
-<wire x1="68.58" y1="104.14" x2="86.36" y2="104.14" width="0.1524" layer="91"/>
-<junction x="86.36" y="104.14"/>
-<wire x1="86.36" y1="104.14" x2="101.6" y2="104.14" width="0.1524" layer="91"/>
-<pinref part="U$7" gate="G$1" pin="GND"/>
-<junction x="86.36" y="104.14"/>
 <junction x="101.6" y="104.14"/>
 <pinref part="B2" gate="G$1" pin="-"/>
@@
 <wire x1="129.54" y1="114.3" x2="129.54" y2="104.14" width="0.1524" layer="91"/>
 <wire x1="101.6" y1="104.14" x2="129.54" y2="104.14" width="0.1524" layer="91"/>
-<label x="96.52" y="104.14" size="1.778" layer="95" rot="R270" xref="yes"/>
-<pinref part="C4" gate="G$1" pin="2"/>
-<wire x1="68.58" y1="109.22" x2="68.58" y2="104.14" width="0.1524" layer="91"/>
-<pinref part="C5" gate="G$1" pin="-"/>
+<pinref part="C3" gate="G$1" pin="-"/>
 <wire x1="101.6" y1="109.22" x2="101.6" y2="104.14" width="0.1524" layer="91"/>
-</segment>
-</net>
-<net name="REOUT" class="1">
-<segment>
-<label x="66.04" y="119.38" size="1.778" layer="95"/>
-<wire x1="68.58" y1="119.38" x2="67.31" y2="119.38" width="0.1524" layer="91"/>
-<pinref part="D2" gate="G$1" pin="+"/>
-<pinref part="U$7" gate="G$1" pin="VOUT"/>
-<wire x1="73.66" y1="119.38" x2="68.58" y2="119.38" width="0.1524" layer="91"/>
-<junction x="68.58" y="119.38"/>
-<pinref part="C4" gate="G$1" pin="1"/>
-<wire x1="68.58" y1="116.84" x2="68.58" y2="119.38" width="0.1524" layer="91"/>
+<pinref part="C4" gate="G$1" pin="-"/>
+<wire x1="66.04" y1="109.22" x2="66.04" y2="104.14" width="0.1524" layer="91"/>
+<wire x1="66.04" y1="104.14" x2="83.82" y2="104.14" width="0.1524" layer="91"/>
+<wire x1="83.82" y1="104.14" x2="83.82" y2="110.49" width="0.1524" layer="91"/>
+<junction x="83.82" y="104.14"/>
+<pinref part="U2" gate="G$1" pin="GND"/>
+<wire x1="83.82" y1="104.14" x2="101.6" y2="104.14" width="0.1524" layer="91"/>
+<label x="83.82" y="104.14" size="1.778" layer="95" rot="R270" xref="yes"/>
 </segment>
 </net>
@@
 <pinref part="B2" gate="G$1" pin="+"/>
 <wire x1="109.22" y1="114.3" x2="116.84" y2="114.3" width="0.1524" layer="91"/>
-<pinref part="U$7" gate="G$1" pin="VIN"/>
-<wire x1="101.6" y1="119.38" x2="99.06" y2="119.38" width="0.1524" layer="91"/>
 <junction x="101.6" y="119.38"/>
-<pinref part="C5" gate="G$1" pin="+"/>
+<pinref part="C3" gate="G$1" pin="+"/>
 <wire x1="101.6" y1="116.84" x2="101.6" y2="119.38" width="0.1524" layer="91"/>
+<pinref part="U2" gate="G$1" pin="IN"/>
+<wire x1="101.6" y1="119.38" x2="95.25" y2="119.38" width="0.1524" layer="91"/>
 </segment>
 </net>
@@
 <label x="55.88" y="119.38" size="1.778" layer="95" rot="R180" xref="yes"/>
 <pinref part="D2" gate="G$1" pin="-"/>
-<wire x1="59.69" y1="119.38" x2="55.88" y2="119.38" width="0.1524" layer="91"/>
+<wire x1="57.15" y1="119.38" x2="55.88" y2="119.38" width="0.1524" layer="91"/>
 </segment>
 <segment>
@@
 </segment>
 </net>
+<net name="N$2" class="0">
+<segment>
+<pinref part="U2" gate="G$1" pin="OUT"/>
+<pinref part="D2" gate="G$1" pin="+"/>
+<wire x1="72.39" y1="119.38" x2="66.04" y2="119.38" width="0.1524" layer="91"/>
+<pinref part="C4" gate="G$1" pin="+"/>
+<wire x1="66.04" y1="119.38" x2="64.77" y2="119.38" width="0.1524" layer="91"/>
+<wire x1="66.04" y1="116.84" x2="66.04" y2="119.38" width="0.1524" layer="91"/>
+<junction x="66.04" y="119.38"/>
+</segment>
+</net>

Commit message: Renumber parts/reversion
Parts:
- removed J4: (no value), dp_devices:CON_DC_M-DC_SMD
- added J3: 4P-SMD-2.0-90D, Seeed-OPL-Connector:GROVE-CONNECTOR-SMD-90D(4+2P-2.0)
- C1: value 1µF -> 10uF; device microbuilder:CAP_CERAMIC0603 -> adafruit:CPOL-US153CLV-0405
- C2: value 1µF -> 100uF 50V; device microbuilder:CAP_CERAMIC0603 -> adafruit:CPOL-US153CLV-0810
- C3: value 100uF 50V -> 1µF; device adafruit:CPOL-US153CLV-0810 -> microbuilder:CAP_CERAMIC0603
- C4: value 10uF -> 1µF; device adafruit:CPOL-US153CLV-0405 -> microbuilder:CAP_CERAMIC0603
- J1: value 4P-SMD-2.0-90D -> (none); device Seeed-OPL-Connector:GROVE-CONNECTOR-SMD-90D(4+2P-2.0) -> dp_devices:CON_DC_M-DC_SMD
- R1: value 10K -> 100K; device microbuilder:RESISTOR0603 -> resistor:R-EU_R0603
- R2: device microbuilder:RESISTOR0603 -> resistor:R-EU_R0603
- R5: value 100R -> 10K
- R6: value 100K -> 100R; device resistor:R-EU_R0603 -> microbuilder:RESISTOR0603
- R8: device resistor:R-EU_R0603 -> microbuilder:RESISTOR0603
- U1: value ADS1115IDGST -> SR05; device microbuilder:ADC_ADS1015 -> Seeed-OPL-ic:PMIC-L7805CV-DG(TO-220)ALT
- U2: value SR05 -> ADS1115IDGST; device Seeed-OPL-ic:PMIC-L7805CV-DG(TO-220)ALT -> microbuilder:ADC_ADS1015
- renumbered 0X48 to 0X1, 0X49 to 0X2, B2 to B1, D2 to D1
Connections:
- net 3V: now also C4.P$1, J3.3; no longer C2.P$1, J1.3
- net ADDR: now also R8.1, U2.ADDR; no longer R3.1, U1.ADDR
- net AGND: now also C1.-, C2.-, C4.P$2, J3.4, U1.GND; no longer C2.P$2, C3.-, C4.-, J1.4, U2.GND
- net AIN0: now also J1.P1, R2.2, U2.AIN0; no longer J4.P1, R7.2, U1.AIN0
- net AIN1: now also R1.2, R2.1; no longer R6.2, R8.1
- net AIN2: now also R6.1, U2.AIN2; no longer R5.1, U1.AIN2
- net AIN3: now also R6.2, U2.AIN3; no longer R5.2, U1.AIN3
- net ALERT: now also R5.2, U2.ALERT; no longer R4.2, U1.ALERT
- net GND: now also C3.P$1, J3.SS1, J3.SS2, R8.2, U2.GND; no longer C1.P$1, J1.SS1, J1.SS2, R3.2, U1.GND
- net N$1: now also R7.2, U2.AIN1; no longer R8.2, U1.AIN1
- net N$2: now also C1.+, U1.OUT; no longer C4.+, U2.OUT
- net N$3: now also J1.P2, R1.1; no longer J4.P2, R6.1
- net N$4: now also C2.+, U1.IN; no longer C3.+, U2.IN
- net SCL: now also J3.1, R3.2, U2.SCL; no longer J1.1, R1.2, U1.SCL
- net SDA: now also J3.2, R4.2, U2.SDA; no longer J1.2, R2.2, U1.SDA
- net VDD: now also C3.P$2, R3.1, R5.1, U2.VDD; no longer C1.P$2, R1.1, R2.1, U1.VDD
Other:
- moved on the sheet: R1, R2, R3, R4, R5, R6, R7, R8
