File: ADS1115_Featherwing.sch (EAGLE design)
At the start: 26 parts, among them J2 ST-PJ-312, J3 4P-SMD-2.0-90D, U1 SR05, U2 ADS1115IDGST

Commit message: Rewired with better net names
Parts:
- R7: device resistor:R-EU_R0603 -> microbuilder:RESISTOR0603
- renumbered 0X1 to 0X48, 0X2 to 0X49
Connections:
- removed net AIN0: B1.AC2, J1.P1, R2.2, U2.AIN0
- removed net AIN1: R1.2, R2.1, R7.1
- removed net AIN2: J2.COM1, R6.1, U2.AIN2
- removed net AIN3: J2.L, R6.2, U2.AIN3
- new net I_AC+: J2.COM1, R6.1, U2.AIN0
- new net I_AC-: J2.L, R6.2, U2.AIN1
- new net V_AC+: R1.2, R2.1, U2.AIN3
- new net V_AC-: B1.AC2, J1.P1, R2.2, R7.1
- net AGND: now also J3.SS1, J3.SS2
- net GND: no longer J3.SS1, J3.SS2
- net N$1: now also U2.AIN2; no longer U2.AIN1
Other:
- moved on the sheet: R7

Commit message: Added clamper and power LED
Parts:
- added C5, C6, C7, C8: 33nF, microbuilder:CAP_CERAMIC0603
- added PWR: GREEN, Discrete-new:LED'0603'
- added R10, R13, R9: 1K, microbuilder:RESISTOR0603
- added R11: 10K, microbuilder:RESISTOR0603
- added R12: VARISTORCN0603, varistor:VARISTORCN0603
- added R14: 1k, Discrete-new:RES-0603
- R7: value 10K -> 1K
- R8: value 10K -> VARISTORCN0603; device microbuilder:RESISTOR0603 -> varistor:VARISTORCN0603
Connections:
- new net N$5: C5.P$1, R7.2, R8.1, U2.AIN0
- new net N$6: C7.P$1, R10.2, R12.1, U2.AIN2
- new net N$7: C8.P$2, R12.2, R13.2, U2.AIN3
- new net N$8: PWR.+, R14.2
- net ADDR: now also R11.1; no longer R8.1
- net AGND: now also PWR.-
- net GND: now also C5.P$2, C6.P$1, C7.P$2, C8.P$1, R11.2; no longer R8.2
- net I_AC+: now also R10.1; no longer U2.AIN0
- net I_AC-: now also R13.1; no longer U2.AIN1
- net N$1: now also C6.P$2, R8.2, R9.2, U2.AIN1; no longer R7.2, U2.AIN2
- net USB: now also R14.1
- net V_AC+: now also R7.1; no longer U2.AIN3
- net V_AC-: now also R9.1; no longer R7.1
Other:
- moved on the sheet: R7

Commit message: Reposition parts
Parts:
- R1: value 100K -> 120K
Changed lines of the file:
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@@
 <part name="FRAME1" library="SparkFun-Aesthetics" deviceset="FRAME-A4L" device=""/>
 <part name="MS1" library="adafruit" deviceset="FEATHERWING" device=""/>
-<part name="R1" library="resistor" deviceset="R-EU_" device="R0603" value="100K"/>
+<part name="R1" library="resistor" deviceset="R-EU_" device="R0603" value="120K"/>
 <part name="R2" library="resistor" deviceset="R-EU_" device="R0603" value="10K"/>
 <part name="B1" library="rectifier" deviceset="MB*S" device="" technology="8"/>

Commit message: Flipped V_AC pins
Connections:
- net V_AC+: now also B1.AC2, J1.P1, R2.2; no longer R1.2, R2.1
- net V_AC-: now also R1.2, R2.1; no longer B1.AC2, J1.P1, R2.2
Changed lines of the file:
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@@
 <?xml version="1.0" encoding="utf-8"?>
 <!DOCTYPE eagle SYSTEM "eagle.dtd">
-<eagle version="7.4.0">
+<eagle version="7.1.0">
 <drawing>
 <settings>
@@
 <attributes>
 <attribute name="CNAME" value="EMON_FEATHERWING"/>
-<attribute name="CREVISION" value="V3"/>
+<attribute name="CREVISION" value="V4"/>
 <attribute name="DESIGNER" value="@whatnick"/>
 </attributes>
@@
 <net name="V_AC+" class="0">
 <segment>
-<pinref part="R2" gate="G$1" pin="1"/>
-<pinref part="R1" gate="G$1" pin="2"/>
-<wire x1="139.7" y1="111.76" x2="139.7" y2="114.3" width="0.1524" layer="91"/>
-<wire x1="139.7" y1="114.3" x2="139.7" y2="116.84" width="0.1524" layer="91"/>
-<wire x1="139.7" y1="114.3" x2="134.62" y2="114.3" width="0.1524" layer="91"/>
-<junction x="139.7" y="114.3"/>
-<label x="132.08" y="114.3" size="1.778" layer="95"/>
-</segment>
-<segment>
 <pinref part="R7" gate="G$1" pin="1"/>
 <wire x1="10.16" y1="58.42" x2="5.08" y2="58.42" width="0.1524" layer="91"/>
 <label x="5.08" y="58.42" size="1.016" layer="95" rot="R180" xref="yes"/>
 </segment>
-</net>
-<net name="V_AC-" class="1">
 <segment>
 <wire x1="149.86" y1="111.76" x2="149.86" y2="101.6" width="0.1524" layer="91"/>
@@
 <pinref part="J1" gate="J" pin="P1"/>
 </segment>
+</net>
+<net name="V_AC-" class="1">
 <segment>
 <pinref part="R9" gate="G$1" pin="1"/>
@@
 <label x="5.08" y="43.18" size="1.016" layer="95" rot="R180" xref="yes"/>
 </segment>
-</net>
+<segment>
+<pinref part="R2" gate="G$1" pin="1"/>
+<pinref part="R1" gate="G$1" pin="2"/>
+<wire x1="139.7" y1="111.76" x2="139.7" y2="114.3" width="0.1524" layer="91"/>
+<wire x1="139.7" y1="114.3" x2="139.7" y2="116.84" width="0.1524" layer="91"/>
+<wire x1="139.7" y1="114.3" x2="134.62" y2="114.3" width="0.1524" layer="91"/>
+<junction x="139.7" y="114.3"/>
+<label x="132.08" y="114.3" size="1.778" layer="95"/>
+</segment>
+</net>
